Commit message: urdf for PR2 Lite head

File: pr2lite_urdf/config/pr2lite_head.xacro (robot description, xacro)
@@ -9,11 +9,4 @@
 >
     <!-- Included URDF Files -->
-    <!--
-     From Matthew:
-      width of outer torso: 0.526999 meters
-      height of outer torso: 0.771906 meters
-      width of joints of arms: 0.4126992 meters
-      joints of arms: 0.05715
-    -->
     <include filename="$(find erratic_description)/urdf/materials.urdf.xacro" />
     <include filename="$(find erratic_description)/urdf/erratic_computer.xacro" />
@@ -35,5 +28,5 @@
     <property name="inner_torso_bottom_size_z" value="0.3" />
     <property name="inner_torso_top_size_x" value="0.17" />
-    <property name="inner_torso_top_size_y" value="0.4953" />
+    <property name="inner_torso_top_size_y" value="0.48" />
     <property name="inner_torso_top_size_z" value="0.46" />
     <property name="wheel_radius" value="0.0762" />
@@ -49,5 +42,6 @@
     <property name="z1" value="0.21844" />
     <property name="shelf_width" value="0.00635" />
-        <!-- base_footprint is a fictitious link(frame) that is on the ground right below base_link origin, navigation stack depends on this frame -->
+        <!-- base_footprint is a fictitious link(frame) that is on the ground right below base_link origin,
+             navigation stack depends on this frame -->
         <link name="base_footprint">
             <inertial>
@@ -59,5 +53,5 @@
             </inertial>
             <visual>
-	        <origin xyz="0.0 0.0 ${base_size_z/2 + caster_width}" rpy="0 0 0" />
+	    <origin xyz="0.0 0.0 ${base_size_z/2 + caster_width}" rpy="0 0 0" />
                 <geometry>
                     <box size="0.001 0.001 0.001" />
@@ -103,5 +97,5 @@
         </link>
         <joint name="base_inner_torso_joint" type="fixed">
-            <origin xyz="${inner_torso_bottom_size_x/2-base_size_x/2} 0.0 ${inner_torso_bottom_size_z/2+base_size_z}"/>
+            <origin xyz="${inner_torso_bottom_size_x/2-(base_size_x/2)} 0.0 ${inner_torso_bottom_size_z/2+base_size_z}"/>
             <parent link="base_link"/>
             <child link="inner_torso_bottom_link" />
@@ -109,5 +103,5 @@
         <link name="inner_torso_bottom_link">
             <inertial>
-                <mass value="0" />
+                <mass value="20" />
                 <origin xyz="0.0 0.0 0.0" />
                 <inertia ixx="1.0" ixy="0.0" ixz="0.0"
@@ -129,5 +123,5 @@
             </collision>
         </link>
-        <!-- 6.85in x 19 x 17.9 -->
+        <!-- 6.85in x 19 x 17.9 -->`
         <joint name="inner_torso_top_joint" type="fixed">
             <origin xyz="${-inner_torso_bottom_size_x/2 + inner_torso_top_size_x/2} 0.0 0.0" rpy="0 0 0" />
@@ -137,5 +131,5 @@
         <link name="inner_torso_top_link">
             <inertial>
-                <mass value="0" />
+                <mass value="20" />
                 <origin xyz="${-inner_torso_top_size_x/2 + inner_torso_top_size_x/2} 0.0 0.0" />
                 <inertia ixx="1.0" ixy="0.0" ixz="0.0"
@@ -163,11 +157,4 @@
 </joint>
 <link name="torso_lift_link">
-            <inertial>
-                <mass value="0" />
-                <origin xyz="0.0 0.0 0.0" />
-                <inertia ixx="1.0" ixy="0.0" ixz="0.0"
-                         iyy="1.0" iyz="0.0"
-                         izz="1.0" />
-            </inertial>
   <visual>
     <axis xyz="0 0 0" />
@@ -186,11 +173,4 @@
 </joint>
 <link name="torso_link">
-           <inertial>
-                <mass value="0" />
-                <origin xyz="0.0 0.0 0.0" />
-                <inertia ixx="1.0" ixy="0.0" ixz="0.0"
-                         iyy="1.0" iyz="0.0"
-                         izz="1.0" />
-            </inertial>
   <visual>
     <axis xyz="0 0 0" />
@@ -206,11 +186,4 @@
 </joint>
 <link name="bottom_outer_torso_link">
-            <inertial>
-                <mass value="0" />
-                <origin xyz="0.0 0.0 0.0" />
-                <inertia ixx="1.0" ixy="0.0" ixz="0.0"
-                         iyy="1.0" iyz="0.0"
-                         izz="1.0" />
-            </inertial>
   <visual>
     <axis xyz="0 0 0" />
@@ -226,11 +199,4 @@
 </joint>
 <link name="top_shelf_link">
-            <inertial>
-                <mass value="0" />
-                <origin xyz="0.0 0.0 0.0" />
-                <inertia ixx="1.0" ixy="0.0" ixz="0.0"
-                         iyy="1.0" iyz="0.0"
-                         izz="1.0" />
-            </inertial>
   <visual>
     <origin xyz="${-inch_to_meter*2.5} ${inch_to_meter*0} ${inch_to_meter*30.5/2}" rpy="0 0 0"/>
@@ -243,18 +209,11 @@
   <parent link="top_shelf_link"/>
   <child link="neck_link"/>
-  <origin xyz="${inch_to_meter*(-3+(.25/2))} ${inch_to_meter*0} ${inch_to_meter*(15.25)}" rpy="0 0 0"/>
+  <origin xyz="${inch_to_meter*0} ${inch_to_meter*7} ${inch_to_meter*(15-3)}" rpy="0 0 0"/>
 </joint>
 <link name="neck_link">
-            <inertial>
-                <mass value="0" />
-                <origin xyz="0.0 0.0 0.0" />
-                <inertia ixx="1.0" ixy="0.0" ixz="0.0"
-                         iyy="1.0" iyz="0.0"
-                         izz="1.0" />
-            </inertial>
-  <visual>
-    <origin xyz="${inch_to_meter*0} ${inch_to_meter*0} ${inch_to_meter*6.5/2}" rpy="0 0 0"/>
-    <geometry><box size="${inch_to_meter*-.25} ${inch_to_meter*5.75} ${inch_to_meter*6.5}"/></geometry>
-    <material name="red"><color rgba="0 0.9 0.9 1.0"/></material>
+  <visual>
+    <origin xyz="${inch_to_meter*0} ${inch_to_meter*0} ${inch_to_meter*0}" rpy="0 0 0"/>
+    <geometry><box size="${inch_to_meter*6.5} ${inch_to_meter*5.75} ${inch_to_meter*.25}"/></geometry>
+    <material name="Silver1"><color rgba="0 0.9 0.9 1.0"/></material>
   </visual>
 </link>
@@ -262,39 +221,35 @@
   <parent link="neck_link"/>
   <child link="top_neck_link"/>
-  <origin xyz="${inch_to_meter*0} ${inch_to_meter*0} ${inch_to_meter*(6.5)}" rpy="0 0 0"/>
+  <origin xyz="${inch_to_meter*0} ${inch_to_meter*0} ${inch_to_meter*(15-3)}" rpy="0 0 0"/>
 </joint>
 <link name="top_neck_link">
-            <inertial>
-                <mass value="0" />
-                <origin xyz="0.0 0.0 0.0" />
-                <inertia ixx="1.0" ixy="0.0" ixz="0.0"
-                         iyy="1.0" iyz="0.0"
-                         izz="1.0" />
-            </inertial>
-  <visual>
-    <origin xyz="${inch_to_meter*2} ${inch_to_meter*0} ${inch_to_meter*.25/2}" rpy="0 0 0"/>
-    <geometry><box size="${inch_to_meter*4} ${inch_to_meter*5.75} ${inch_to_meter*.25}"/></geometry>
+  <visual>
+    <origin xyz="${inch_to_meter*0} ${inch_to_meter*0} ${inch_to_meter*0}" rpy="0 0 0"/>
+    <geometry><box size="${inch_to_meter*.25} ${inch_to_meter*5.75} ${inch_to_meter*4}"/></geometry>
+    <material name="Silver1"><color rgba="0 0.9 0.9 1.0"/></material>
+  </visual>
+</link>
+<joint name="neck_head_joint" type="revolute">
+  <parent link="top_neck_link"/>
+  <child link="head_pan_link"/>
+  <origin xyz="${inch_to_meter*0} ${inch_to_meter*(-2.875)} ${inch_to_meter*(-2)}" rpy="0 0 0"/>
+</joint>
+<link name="head_pan_link">
+  <visual>
+    <origin xyz="${inch_to_meter*0} ${inch_to_meter*0} ${inch_to_meter*0}" rpy="0 0 0"/>
+    <geometry><box size="${inch_to_meter*4} ${inch_to_meter*.25} ${inch_to_meter*4}"/></geometry>
     <material name="Silver1"><color rgba="0 0.9 0.9 1.0"/></material>
   </visual>
 </link>
 <!-- 4x 13.14 -->
-<joint name="head_base_joint" type="revolute">
-  <limit effort="10" lower="-3.1416" upper="3.1416" velocity="3"/>
-  <parent link="top_neck_link"/>
+<joint name="neck_head_joint" type="revolute">
+  <parent link="head_pan_link"/>
   <child link="head_base_link"/>
-  <origin xyz="${inch_to_meter*2} ${inch_to_meter*(0)} ${inch_to_meter*(.25+.125)}" rpy="0 0 0"/>
-  <axis xyz="0 0 1"/>
+  <origin xyz="${inch_to_meter*0} ${inch_to_meter*(-2.875)} ${inch_to_meter*(-2)}" rpy="0 0 0"/>
 </joint>
 <link name="head_base_link">
-            <inertial>
-                <mass value="0" />
-                <origin xyz="0.0 0.0 0.0" />
-                <inertia ixx="1.0" ixy="0.0" ixz="0.0"
-                         iyy="1.0" iyz="0.0"
-                         izz="1.0" />
-            </inertial>
-  <visual>
-    <origin xyz="${inch_to_meter*0} ${inch_to_meter*0} ${inch_to_meter*0}" rpy="0 0 0"/>
-    <geometry><box size="${inch_to_meter*4} ${inch_to_meter*13.14} ${inch_to_meter*.25}"/></geometry>
+  <visual>
+    <origin xyz="${inch_to_meter*0} ${inch_to_meter*0} ${inch_to_meter*0}" rpy="0 0 0"/>
+    <geometry><box size="${inch_to_meter*.25} ${inch_to_meter*13.14} ${inch_to_meter*4}"/></geometry>
     <material name="Silver1"><color rgba="0 0.9 0.9 1.0"/></material>
   </visual>
@@ -303,201 +258,39 @@
   <parent link="head_base_link"/>
   <child link="head_side_link"/>
-  <origin xyz="${inch_to_meter*0} ${inch_to_meter*((13.14/2)-(.25/2))} ${inch_to_meter*(2.5)}" rpy="0 0 0"/>
+  <origin xyz="${inch_to_meter*0} ${inch_to_meter*(0.)} ${inch_to_meter*((13.14 -.25)/2)}" rpy="0 0 0"/>
 </joint>
 <link name="head_side_link">
-            <inertial>
-                <mass value="0" />
-                <origin xyz="0.0 0.0 0.0" />
-                <inertia ixx="1.0" ixy="0.0" ixz="0.0"
-                         iyy="1.0" iyz="0.0"
-                         izz="1.0" />
-            </inertial>
-  <visual>
-    <origin xyz="${inch_to_meter*0} ${inch_to_meter*(-.25/2)} ${inch_to_meter*0}" rpy="0 0 0"/>
-    <geometry><box size="${inch_to_meter*4} ${inch_to_meter*.25} ${inch_to_meter*5}"/></geometry>
+  <visual>
+    <origin xyz="${inch_to_meter*0} ${inch_to_meter*0} ${inch_to_meter*0}" rpy="0 0 0"/>
+    <geometry><box size="${inch_to_meter*5} ${inch_to_meter*.25} ${inch_to_meter*4}"/></geometry>
     <material name="Silver1"><color rgba="0 0.9 0.9 1.0"/></material>
   </visual>
 </link>
 <joint name="head_tilt_joint" type="revolute">
-  <limit effort="10" lower="-3.1416" upper="3.1416" velocity="3"/>
   <parent link="head_side_link"/>
   <child link="kinect_side_link"/>
-  <origin xyz="${inch_to_meter*0} ${inch_to_meter*(-.25)} ${inch_to_meter*.5}" rpy="0 0 0"/>
-  <axis xyz="0 1 0"/>
+  <origin xyz="${inch_to_meter*0} ${inch_to_meter*(3)} ${inch_to_meter*(0)}" rpy="0 0 0"/>
 </joint>
 <link name="kinect_side_link">
-            <inertial>
-                <mass value="0" />
-                <origin xyz="0.0 0.0 0.0" />
-                <inertia ixx="1.0" ixy="0.0" ixz="0.0"
-                         iyy="1.0" iyz="0.0"
-                         izz="1.0" />
-            </inertial>
-  <visual>
-    <origin xyz="${inch_to_meter*0} ${inch_to_meter*(-.25/2)} ${inch_to_meter*0}" rpy="0 0 0"/>
-    <geometry><box size="${inch_to_meter*(4)} ${inch_to_meter*-.25} ${inch_to_meter*(4)}"/></geometry>
-    <material name="green"><color rgba="0 0.9 0.9 1.0"/></material>
-  </visual>
-</link>
-<joint name="kinect_side_joint" type="fixed">
+  <visual>
+    <origin xyz="${inch_to_meter*0} ${inch_to_meter*0} ${inch_to_meter*0}" rpy="0 0 0"/>
+    <geometry><box size="${inch_to_meter*(3.54 -.21} ${inch_to_meter*.25} ${inch_to_meter*4}"/></geometry>
+    <material name="Silver1"><color rgba="0 0.9 0.9 1.0"/></material>
+  </visual>
+</link>
+<joint name="kinect_side_link" type="fixed">
   <parent link="kinect_side_link"/>
   <child link="kinect_base_link"/>
-  <origin xyz="${inch_to_meter*-(0)} ${inch_to_meter*(0)} ${inch_to_meter*-(2.04+(.25/2))}" rpy="0 0 0"/>
+  <origin xyz="${inch_to_meter*-(3.54 -.21)} ${inch_to_meter*(0)} ${inch_to_meter*(0)}" rpy="0 0 0"/>
 </joint>
 <link name="kinect_base_link">
-            <inertial>
-                <mass value="0" />
-                <origin xyz="0.0 0.0 0.0" />
-                <inertia ixx="1.0" ixy="0.0" ixz="0.0"
-                         iyy="1.0" iyz="0.0"
-                         izz="1.0" />
-           </inertial>
-  <visual>
-    <origin xyz="${inch_to_meter*0} ${inch_to_meter*(-11.5/2)} ${inch_to_meter*0}" rpy="0 0 0"/>
-    <geometry><box size="${inch_to_meter*4} ${inch_to_meter*11.5} ${inch_to_meter*-.25}"/></geometry>
-    <material name="Green"><color rgba="0 0.9 0.9 1.0"/></material>
-  </visual>
-</link>
-<!-- KINECT STANDOFF -->
-<property name="M_SCALE" value="0.001"/>
-    <joint name="standoff1_kinect_joint" type="fixed">
-      <origin xyz="${inch_to_meter*11/16} ${inch_to_meter*-1.75} ${inch_to_meter*0}" rpy="0 0 0" />
-      <parent link="kinect_base_link" />
-      <child link="standoff1_kinect_link" />
-    </joint>
-    <link name="standoff1_kinect_link">
-      <inertial>
-        <mass value="0.001" />
-        <origin xyz="0 0 0" />
-        <inertia ixx="0.0001" ixy="0.0" ixz="0.0"
-          iyy="0.0001" iyz="0.0"
-          izz="0.0001" />
-      </inertial>
-      <visual>
-        <origin xyz=" 0 0 0 " rpy="0 0 0" />
-        <geometry>
-          <mesh filename="package://pr2lite_urdf/config/meshes/68-04556-RA_Kinect_Standoff_Assy.3ds" scale="${M_SCALE} ${M_SCALE} ${M_SCALE}"/>
-        </geometry>
-      </visual>
-      <collision>
-        <origin xyz="0.0 0.0 0.0" rpy="0 0 0" />
-        <geometry>
-          <cylinder length="0.008585" radius="0.001111"/>
-        </geometry>
-      </collision>
-    </link>
-    <joint name="standoff2_kinect_joint" type="fixed">
-      <origin xyz="${inch_to_meter*11/16} ${inch_to_meter*(-1.75-7.75)} ${inch_to_meter*0}" rpy="0 0 0" />
-      <parent link="kinect_base_link" />
-      <child link="standoff2_kinect_link" />
-    </joint>
-    <link name="standoff2_kinect_link">
-      <inertial>
-        <mass value="0.001" />
-        <origin xyz="0 0 0" />
-        <inertia ixx="0.0001" ixy="0.0" ixz="0.0"
-          iyy="0.0001" iyz="0.0"
-          izz="0.0001" />
-      </inertial>
-      <visual>
-        <origin xyz=" 0 0 0 " rpy="0 0 0" />
-        <geometry>
-          <mesh filename="package://pr2lite_urdf/config/meshes/68-04556-RA_Kinect_Standoff_Assy.3ds" scale="${M_SCALE} ${M_SCALE} ${M_SCALE}"/>
-        </geometry>
-      </visual>
-      <collision>
-        <origin xyz="0.0 0.0 0.0" rpy="0 0 0" />
-        <geometry>
-          <cylinder length="0.008585" radius="0.001111"/>
-        </geometry>
-      </collision>
-    </link>
-<!-- KINECT SENSOR -->
-<joint name="base_kinect_joint" type="fixed">
-<!--
-      <origin xyz="-0.0844382 0 0.1047496" rpy="0 0 0" />
-    <origin xyz="${inch_to_meter*11/16} ${inch_to_meter*(-11.5/2)} ${0.1047496}" rpy="0 0 0"/>
--->
-    <origin xyz="${inch_to_meter*(1+3/8)} ${inch_to_meter*(-11.5/2)} ${0.1047496}" rpy="0 0 0"/>
-      <parent link="kinect_base_link" />
-      <child link="kinect_link" />
-    </joint>
-    <link name="kinect_link">
-      <inertial>
-        <mass value="12" />
-        <origin xyz="0 0 0" />
-        <inertia ixx="1.0" ixy="0.0" ixz="0.0"
-                 iyy="1.0" iyz="0.0"
-                 izz="1.0" />
-      </inertial>
-      <visual>
-        <origin xyz=" 0 0 0 " rpy="0 0 0" />
-        <geometry>
-          <mesh filename="package://pr2lite_urdf/config/meshes/68-04546_Kinect_Sensor.3ds" scale="${M_SCALE} ${M_SCALE} ${M_SCALE}"/>
-        </geometry>
-      </visual>
-      <collision>
-        <origin xyz="0.0 0.0 0.0" rpy="0 0 0" />
-        <geometry>
-          <mesh filename="package://pr2lite_urdf/config/meshes/68-04546_Kinect_Sensor.3ds"/>
-          </geometry>
-      </collision>
-    </link>
-    <joint name="kinect_depth_joint" type="fixed">
-      <origin xyz="0 0.018 0" rpy="0 0 0" />
-      <parent link="kinect_link" />
-      <child link="kinect_depth_frame" />
-    </joint>
-    <link name="kinect_depth_frame">
-      <inertial>
-        <mass value="0.0001" />
-        <origin xyz="0 0 0" />
-        <inertia ixx="0.0001" ixy="0.0" ixz="0.0"
-                 iyy="0.0001" iyz="0.0"
-                 izz="0.0001" />
-      </inertial>
-    </link>
-    <joint name="kinect_depth_optical_joint" type="fixed">
-      <origin xyz="0 0 0" rpy="${-M_PI/2} 0 ${-M_PI/2}" />
-      <parent link="kinect_depth_frame" />
-      <child link="kinect_depth_optical_frame" />
-    </joint>
-    <link name="kinect_depth_optical_frame">
-      <inertial>
-        <mass value="0.0001" />
-        <origin xyz="0 0 0" />
-        <inertia ixx="0.0001" ixy="0.0" ixz="0.0"
-                 iyy="0.0001" iyz="0.0"
-                 izz="0.0001" />
-      </inertial>
-    </link>
-    <joint name="kinect_rgb_joint" type="fixed">
-      <origin xyz="0 -0.005 0" rpy="0 0 0" />
-      <parent link="kinect_link" />
-      <child link="kinect_rgb_frame" />
-    </joint>
-    <link name="kinect_rgb_frame">
-      <inertial>
-        <mass value="0.0001" />
-        <origin xyz="0 0 0" />
-        <inertia ixx="0.0001" ixy="0.0" ixz="0.0"
-                 iyy="0.0001" iyz="0.0"
-                 izz="0.0001" />
-      </inertial>
-    </link>
-    <joint name="kinect_rgb_optical_joint" type="fixed">
-      <origin xyz="0 0 0" rpy="${-M_PI/2} 0 ${-M_PI/2}" />
-      <parent link="kinect_rgb_frame" />
-      <child link="kinect_rgb_optical_frame" />
-    </joint>
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