Commit message: urdf for PR2 Lite head

File: pr2lite_urdf/config/pr2lite_smartarm.xacro (robot description, xacro)
@@ -32,4 +32,7 @@
           <!-- shoulder pan cylindar to lin act joint -->
           <origin xyz="${inch_to_meter*(1.5)} ${inch_to_meter*0} ${inch_to_meter*7.3575}" rpy="0 0 0"/>
+<!--
+          <origin xyz="${inch_to_meter*(.5)} ${inch_to_meter*0} ${inch_to_meter*7.3575}" rpy="0 0 0"/>
+-->
           <parent link="${side}_shoulder_caster_link"/>
           <child link="${side}_lower_linear_actuator_link"/>
@@ -212,12 +215,12 @@
                 <origin xyz="0.0 0.0 0.0" rpy="0 0 0" />
                 <geometry>
-                    <mesh filename="package://smart_arm_description/meshes/arm_base.stl"/>
-                </geometry>
-            </visual>
-<!--
-            <collision>
-                <origin xyz="0.0 0.0 0.0" rpy="0 0 0" />
-                <geometry>
-                    <mesh filename="package://smart_arm_description/meshes/convex/arm_base_convex.stlb"/>
+                    <mesh filename="package://pr2lite_urdf/config/meshes/arm_base.stl"/>
+                </geometry>
+            </visual>
+<!--
+            <collision>
+                <origin xyz="0.0 0.0 0.0" rpy="0 0 0" />
+                <geometry>
+                    <mesh filename="package://pr2lite_urdf/config/meshes/arm_base_convex.stlb"/>
                 </geometry>
             </collision>
@@ -235,12 +238,12 @@
                 <origin xyz="0.0 0.0 0.005" rpy="0 0 0" />
                 <geometry>
-                    <mesh filename="package://smart_arm_description/meshes/arm_shoulder_pan.stl"/>
-                </geometry>
-            </visual>
-<!--
-            <collision>
-                <origin xyz="0.0 0.0 0.0" rpy="0 0 0" />
-                <geometry>
-                    <mesh filename="package://smart_arm_description/meshes/convex/arm_shoulder_pan_convex.stlb"/>
+                    <mesh filename="package://pr2lite_urdf/config/meshes/arm_shoulder_pan.stl"/>
+                </geometry>
+            </visual>
+<!--
+            <collision>
+                <origin xyz="0.0 0.0 0.0" rpy="0 0 0" />
+                <geometry>
+                    <mesh filename="package://pr2lite_urdf/config/meshes/arm_shoulder_pan_convex.stlb"/>
                 </geometry>
             </collision>
@@ -258,12 +261,12 @@
                 <origin xyz="0.0 0.0 0.0" rpy="0 0 0" />
                 <geometry>
-                    <mesh filename="package://smart_arm_description/meshes/arm_shoulder_tilt.stl"/>
-                </geometry>
-            </visual>
-<!--
-            <collision>
-                <origin xyz="0.0 0.0 0.0" rpy="0 0 0" />
-                <geometry>
-                    <mesh filename="package://smart_arm_description/meshes/convex/arm_shoulder_tilt_convex.stlb"/>
+                    <mesh filename="package://pr2lite_urdf/config/meshes/arm_shoulder_tilt.stl"/>
+                </geometry>
+            </visual>
+<!--
+            <collision>
+                <origin xyz="0.0 0.0 0.0" rpy="0 0 0" />
+                <geometry>
+                    <mesh filename="package://pr2lite_urdf/config/meshes/arm_shoulder_tilt_convex.stlb"/>
                 </geometry>
             </collision>
@@ -281,12 +284,12 @@
                 <origin xyz="0.0 0.0 0.0" rpy="0 0 0" />
                 <geometry>
-                    <mesh filename="package://smart_arm_description/meshes/arm_elbow_tilt.stl"/>
-                </geometry>
-            </visual>
-<!--
-            <collision>
-                <origin xyz="0.0 0.0 0.0" rpy="0 0 0" />
-                <geometry>
-                    <mesh filename="package://smart_arm_description/meshes/convex/arm_elbow_tilt_convex.stlb"/>
+                    <mesh filename="package://pr2lite_urdf/config/meshes/arm_elbow_tilt.stl"/>
+                </geometry>
+            </visual>
+<!--
+            <collision>
+                <origin xyz="0.0 0.0 0.0" rpy="0 0 0" />
+                <geometry>
+                    <mesh filename="package://pr2lite_urdf/config/meshes/arm_elbow_tilt_convex.stlb"/>
                 </geometry>
             </collision>
@@ -304,12 +307,12 @@
                 <origin xyz="0.0 0.0 0.0" rpy="0 0 0" />
                 <geometry>
-                    <mesh filename="package://smart_arm_description/meshes/arm_wrist_rotate.stl"/>
-                </geometry>
-            </visual>
-<!--
-            <collision>
-                <origin xyz="0.0 0.0 0.0" rpy="0 0 0" />
-                <geometry>
-                    <mesh filename="package://smart_arm_description/meshes/convex/arm_wrist_rotate_convex.stlb"/>
+                    <mesh filename="package://pr2lite_urdf/config/meshes/arm_wrist_rotate.stl"/>
+                </geometry>
+            </visual>
+<!--
+            <collision>
+                <origin xyz="0.0 0.0 0.0" rpy="0 0 0" />
+                <geometry>
+                    <mesh filename="package://pr2lite_urdf/config/meshes/arm_wrist_rotate_convex.stlb"/>
                 </geometry>
             </collision>
@@ -327,12 +330,12 @@
                 <origin xyz="0.0 0.0 0.0" rpy="0 0 0" />
                 <geometry>
-                    <mesh filename="package://smart_arm_description/meshes/arm_right_finger.stl"/>
-                </geometry>
-            </visual>
-<!--
-            <collision>
-                <origin xyz="0.0 0.0 0.0" rpy="0 0 0" />
-                <geometry>
-                    <mesh filename="package://smart_arm_description/meshes/convex/arm_right_finger_convex.stlb"/>
+                    <mesh filename="package://pr2lite_urdf/config/meshes/arm_right_finger.stl"/>
+                </geometry>
+            </visual>
+<!--
+            <collision>
+                <origin xyz="0.0 0.0 0.0" rpy="0 0 0" />
+                <geometry>
+                    <mesh filename="package://pr2lite_urdf/config/meshes/arm_right_finger_convex.stlb"/>
                 </geometry>
             </collision>
@@ -350,12 +353,12 @@
                 <origin xyz="0.0 0.0 0.0" rpy="0 0 0" />
                 <geometry>
-                    <mesh filename="package://smart_arm_description/meshes/arm_left_finger.stl"/>
-                </geometry>
-            </visual>
-<!--
-            <collision>
-                <origin xyz="0.0 0.0 0.0" rpy="0 0 0" />
-                <geometry>
-                    <mesh filename="package://smart_arm_description/meshes/convex/arm_left_finger_convex.stlb"/>
+                    <mesh filename="package://pr2lite_urdf/config/meshes/arm_left_finger.stl"/>
+                </geometry>
+            </visual>
+<!--
+            <collision>
+                <origin xyz="0.0 0.0 0.0" rpy="0 0 0" />
+                <geometry>
+                    <mesh filename="package://pr2lite_urdf/config/meshes/arm_left_finger_convex.stlb"/>
                 </geometry>
             </collision>
@@ -460,21 +463,29 @@
             <fudgeFactor value="1.0" />
         </gazebo>
+<!--
     <transmission type="pr2_mechanism_model/Pr2LiteShoulderTransmission" name="${side}_pr2lite_shoulder_trans" >
       <actuator       name="${side}_linear_actuator_joint" />
       <gap_joint      name="${side}_shoulder_tilt_joint"
                       />
+-->
       <!-- if a gazebo joint exists as [l|r]_gripper_joint, use this tag to have
            gripper transmission apply torque directly to prismatic joint
            this should be the default behavior in diamondback, deprecating this flag -->
+<!--
       <use_simulated_gripper_joint/>
+-->
       <!-- set passive joint angles so things look nice in rviz -->
+<!--
       <passive_joint  name="${side}_shoulder_tilt_joint"     />
       <passive_joint  name="${side}_lin_act_cyl_joint"     />
       <passive_joint  name="${side}_upper_arm_hinge_joint" />
+-->
       <!-- screw joint to capture gripper "dynamics" -->
+<!--
       <simulated_actuated_joint name="${side}_linear_actuator_joint"
                                 passive_actuated_joint="${side}_gripper_motor_slider_joint"
                                 simulated_reduction="1"   />
     </transmission>
+-->
     </macro>
 </robot>

File: pr2lite_urdf/config/pr2lite_wheel.xacro (robot description, xacro)
@@ -36,4 +36,7 @@
     <property name="motor_block_size_z" value="0.1016"/>
     <property name="wheel_radius" value=".0762"/>
+    <!--
+      from floor to bottom of base is 8.97 inches
+    -->
  <macro name="pr2lite_wheel" params="suffix parent reflect_x reflect_y">
 <!-- * * * Link Definitions * * * -->
